File: circuit diagram/Platine_gijon.sch (EAGLE design)
At the start: 14 parts

Commit message: Electronic working fine and irst circuit diagram
Parts:
- removed JP1, JP2, JP3, JP4, JP5, JP6, JP7, JP8: (no value), jumper:JP1E
- removed R3: 5k, rcl:R-TRIMM3339P
- removed S1: (no value), switch-omron:10-XX
- added C1: 10uF, capacitor-wima:C2,5-3
- added M1: MOTOR, lib_gijon:MOTOR
- added R4: 1k, resistor-power:RAC01
- added S2: (no value), SparkFun-Switches:SWITCH-SPDT-PTH-11.6X4.0MM
- added U1: MD22, lib_gijon:MD22
Connections:
- new net GND: C1.2
- new net N$3: C1.1, R4.2
- new net N$4: R4.1
Other:
- note added: "Input"
- note added: "Output"
- note added: "Poti-Posit."
- note removed: "Motor"
- note removed: "MotorDriver MD22"
- note removed: "Poti-Pos"
- note removed: "Poti-Test"
- moved on the sheet: F1

Commit message: Casi Termino :)
Parts:
- added R3: 1M, resistor-power:RAC01
- added R6: 10k, resistor-power:RAC01
- added U$1: SP200, lib_gijon:SP200
Connections:
- new net 12V: F1.1
- new net 5V: M1.HALL_VCC, R1.E, R2.E, U$1.V+, U1.+5V
- new net N$1: F1.2, U1.MOTOR_+V
- new net N$10: M1.HALL_A_OUT
- new net N$11: M1.HALL_B_OUT
- new net N$2: M1.-MOTOR, U1.MOTOR11
- new net N$5: M1.+MOTOR, U1.MOTOR1
- new net N$6: R1.S, S2.P
- new net N$7: R3.2, R6.1, U$1.INL
- new net N$8: S2.O
- new net N$9: R2.S
- net GND: now also M1.HALL_GND, R1.A, R2.A, R6.2, U$1.GND, U$1.INH, U1.GND, U1.MOTOR_GND
- net N$3: now also U1.SCL
- net N$4: now also R3.1, S2.S
Other:
- note added: "2, ChannelB"
- note added: "3, ChannelA"
- note added: "6, PWM_Output"
- note added: "A0, Input Speed"
- note added: "A3, Poti. - Postion"
- moved on the sheet: B1, C1, F1, R4, S2
